File: src/RPI_Expansion_Board.kicad_sch (KiCad schematic)
At the start: 6 parts, among them J6 USB_C_Receptacle_PowerOnly_6P

Commit message: Begin working on power solution for HDMI + SD
Other:
- sheet GPIO & Low Speed ports: added SD_PWR, SD_PWR_ON; removed none
Changed lines of the file:
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@@
+		)
+	)
+	(global_label "SD_PWR_ON"
+		(shape input)
+		(at 223.52 88.9 180)
+		(fields_autoplaced yes)
+		(effects
+			(font
+				(size 1.27 1.27)
+			)
+			(justify right)
+		)
+		(property "Intersheetrefs" "${INTERSHEET_REFS}"
+			(at 210.1219 88.9 0)
+			(effects
+				(font
+					(size 1.27 1.27)
+				)
+				(justify right)
+				(hide yes)
+			)
+		)
+	)
+	(global_label "SD_PWR"
+		(shape output)
+		(at 223.52 85.09 180)
+		(fields_autoplaced yes)
+		(effects
+			(font
+				(size 1.27 1.27)
+			)
+			(justify right)
+		)
+		(property "Intersheetrefs" "${INTERSHEET_REFS}"
+			(at 213.7505 85.09 0)
+			(effects
+				(font
+					(size 1.27 1.27)
+				)
+				(justify right)
+				(hide yes)
+			)
 		)
 	)
@@
 	)
 	(sheet
-		(at 109.22 76.2)
+		(at 158.75 78.74)
 		(size 46.99 31.75)
 		(fields_autoplaced yes)
@@
 		)
 		(property "Sheetname" "High Speed"
-			(at 109.22 75.4884 0)
+			(at 158.75 78.0284 0)
 			(effects
 				(font
@@
 		)
 		(property "Sheetfile" "highspeed.kicad_sch"
-			(at 109.22 108.5346 0)
+			(at 158.75 111.0746 0)
 			(effects
 				(font
@@
 	)
 	(sheet
-		(at 173.99 76.2)
+		(at 223.52 78.74)
 		(size 38.1 31.75)
 		(fields_autoplaced yes)
@@
 		)
 		(property "Sheetname" "GPIO & Low Speed"
-			(at 173.99 75.4884 0)
+			(at 223.52 78.0284 0)
 			(effects
 				(font
@@
 		)
 		(property "Sheetfile" "gpio_low_speed.kicad_sch"
-			(at 173.99 108.5346 0)
+			(at 223.52 111.0746 0)
 			(effects
 				(font
@@
 			)
 		)
+		(pin "SD_PWR" input
+			(at 223.52 85.09 180)
+			(effects
+				(font
+					(size 1.27 1.27)
+				)
+				(justify left)
+			)
+		)
+		(pin "SD_PWR_ON" output
+			(at 223.52 88.9 180)
+			(effects
+				(font
+					(size 1.27 1.27)
+				)
+				(justify left)
+			)
+		)
